Commit message: feat: ROS 순찰 임무 관리자와 TMC160B 시뮬레이션 추가
- 순찰 Action 인터페이스와 Nav2 임무 관리자 패키지 구현
- 순찰 및 navigation launch에 임무 관리자 연결
- TMC160B 해상도, 시야각, 주기 및 임시 형상 반영

File: src/hazard_guard_simulation/urdf/hazard_guard_m1.urdf.xacro (robot description, xacro)
@@ -27,5 +27,8 @@
   <xacro:property name="base_ground_offset" value="0.0276" />
   <xacro:property name="stock_mass" value="2.74" />
-  <xacro:property name="thermal_mass" value="0.030" />
+  <!-- Provisional TMC160B board-level mass from the current product-family
+       brochure. Verify the delivered enclosure and bracket before the hardware
+       dynamics baseline. -->
+  <xacro:property name="thermal_mass" value="0.052" />
   <xacro:if value="$(arg include_dispenser)">
     <xacro:property
@@ -257,7 +260,8 @@
   </joint>
   <!--
-    TOPDON TC001 provisional front mount. Device geometry and sensor parameters
-    are official; the mounting pose remains a project assumption until the
-    mechanical team supplies its bracket drawing.
+    ThermoEye TMC160B provisional front mount. The 38 x 38 mm board face is
+    based on the manufacturer specification. Board stack depth and the mounting
+    pose remain project assumptions until the delivered unit and bracket are
+    measured.
   -->
   <link name="thermal_camera_link">
@@ -265,10 +269,10 @@
       <mass value="${thermal_mass}" />
       <inertia
-        ixx="0.00001701" ixy="0" ixz="0"
-        iyy="0.00000490" iyz="0"
-        izz="0.00001309" />
+        ixx="0.0000125147" ixy="0" ixz="0"
+        iyy="0.0000071067" iyz="0"
+        izz="0.0000071067" />
     </inertial>
     <visual>
-      <geometry><box size="0.014 0.071 0.042" /></geometry>
+      <geometry><box size="0.014 0.038 0.038" /></geometry>
       <material name="thermal_blue" />
     </visual>
@@ -279,5 +283,5 @@
     </visual>
     <collision>
-      <geometry><box size="0.014 0.071 0.042" /></geometry>
+      <geometry><box size="0.014 0.038 0.038" /></geometry>
     </collision>
   </link>
@@ -437,17 +441,22 @@
     </sensor>
   </gazebo>
-  <!-- Synthetic optical stream only; temperature detections come from the
-       explicitly simulated heat-source node and are never presented as real. -->
+  <!--
+    Synthetic optical stream shaped like the ThermoEye TMC160B:
+      160 x 120 pixels, 57 degree horizontal FOV, nominal 8.7 Hz.
+    The 5 m far clip is a project visualization boundary, not a manufacturer
+    measurement-distance guarantee. Temperature detections come from the
+    explicitly simulated heat-source node and are never presented as real.
+  -->
   <gazebo reference="thermal_camera_link">
     <sensor name="hazard_guard_thermal_camera" type="thermal_camera">
       <always_on>true</always_on>
-      <update_rate>25</update_rate>
+      <update_rate>8.7</update_rate>
       <visualize>${visualize_sensors}</visualize>
       <topic>/thermal_camera</topic>
       <gz_frame_id>thermal_camera_optical_frame</gz_frame_id>
       <camera name="thermal_camera">
-        <horizontal_fov>0.977384381</horizontal_fov>
-        <image><width>256</width><height>192</height><format>L_INT16</format></image>
-        <clip><near>0.1</near><far>5.0</far></clip>
+        <horizontal_fov>0.994837674</horizontal_fov>
+        <image><width>160</width><height>120</height><format>L_INT16</format></image>
+        <clip><near>0.05</near><far>5.0</far></clip>
       </camera>
     </sensor>

Commit message: refactor: ROS 임무 관리자 책임과 센서 설정 분리
- Nav2 통신과 임무 상태 저장을 전용 모듈로 분리
- TMC160B 시뮬레이션 수치를 단일 센서 프로필로 통합
- 상태 저장 테스트와 Python 정적 검사 품질 보강

File: src/hazard_guard_simulation/urdf/hazard_guard_m1.urdf.xacro (robot description, xacro)
@@ -8,7 +8,19 @@
   <xacro:arg name="include_dispenser" default="true" />
   <xacro:arg name="dispenser_mass" default="1.2" />
+  <xacro:arg name="thermal_width" default="160" />
+  <xacro:arg name="thermal_height" default="120" />
+  <xacro:arg name="thermal_update_rate" default="8.7" />
+  <xacro:arg name="thermal_horizontal_fov" default="0.994837674" />
+  <xacro:arg name="thermal_clip_near" default="0.05" />
+  <xacro:arg name="thermal_clip_far" default="5.0" />
   <xacro:property name="simulation_mode" value="$(arg simulation_mode)" />
   <xacro:property name="visualize_sensors" value="$(arg visualize_sensors)" />
   <xacro:property name="dispenser_requested_mass" value="$(arg dispenser_mass)" />
+  <xacro:property name="thermal_width" value="$(arg thermal_width)" />
+  <xacro:property name="thermal_height" value="$(arg thermal_height)" />
+  <xacro:property name="thermal_update_rate" value="$(arg thermal_update_rate)" />
+  <xacro:property name="thermal_horizontal_fov" value="$(arg thermal_horizontal_fov)" />
+  <xacro:property name="thermal_clip_near" value="$(arg thermal_clip_near)" />
+  <xacro:property name="thermal_clip_far" value="$(arg thermal_clip_far)" />
   <!--
     Geometry sources:
@@ -451,12 +463,12 @@
     <sensor name="hazard_guard_thermal_camera" type="thermal_camera">
       <always_on>true</always_on>
-      <update_rate>8.7</update_rate>
+      <update_rate>${thermal_update_rate}</update_rate>
       <visualize>${visualize_sensors}</visualize>
       <topic>/thermal_camera</topic>
       <gz_frame_id>thermal_camera_optical_frame</gz_frame_id>
       <camera name="thermal_camera">
-        <horizontal_fov>0.994837674</horizontal_fov>
-        <image><width>160</width><height>120</height><format>L_INT16</format></image>
-        <clip><near>0.05</near><far>5.0</far></clip>
+        <horizontal_fov>${thermal_horizontal_fov}</horizontal_fov>
+        <image><width>${thermal_width}</width><height>${thermal_height}</height><format>L_INT16</format></image>
+        <clip><near>${thermal_clip_near}</near><far>${thermal_clip_far}</far></clip>
       </camera>
     </sensor>

Commit message: feat(simulation): 열화상 카메라를 RGB-D 옆으로 옮기고 마운트를 인자화
실물에서는 열화상 모듈을 RGB-D 유닛 앞이 아니라 옆이나 위에 붙인다.
위는 불가능하다. LiDAR 스캔 평면이 base_link 기준 z 0.14712 이고 카메라
하우징 윗면이 이미 0.1197 이라, 38 mm 보드를 그 위에 올리면 0.158 까지
올라가 전방 스캔을 가린다.

옆에 두면 보드가 0.087~0.125 에 머물러 스캔 평면 아래로 빠진다. 두 광학
프레임을 x·z 는 같게 두고 y 만 68 mm 벌려, 베이스라인이 순수 횡방향이
되도록 배치한다. 캘리브레이션 결과를 검산하기 가장 쉬운 형태다. 하우징과
4 mm, 차체 옆면보다 6.5 mm 바깥이며 Nav2 풋프린트 반폭 0.155 m 안이다.

마운트 위치와 자세를 xacro 인자로 뺀다. 캘리브레이션이 알려진 오차를
복원하는지 시험하려면 마운트를 의도적으로 틀 수 있어야 한다.

  xacro ... thermal_mount_y:=0.073 thermal_mount_yaw:=0.035

test/test_thermal_mount.py 가 LiDAR 평면 침범, 하우징 겹침, 베이스라인
정렬을 검사한다. 위쪽 마운트 좌표를 넣으면 실패하는 것을 확인했다.

File: src/hazard_guard_simulation/urdf/hazard_guard_m1.urdf.xacro (robot description, xacro)
@@ -14,4 +14,13 @@
   <xacro:arg name="thermal_clip_near" default="0.05" />
   <xacro:arg name="thermal_clip_far" default="5.0" />
+  <!-- Thermal mount, base_link frame. Defaults put the thermal optical frame
+       level with the depth optical frame (x 0.115871, z 0.106136) and 68 mm to
+       its left; see the joint below for why that side. -->
+  <xacro:arg name="thermal_mount_x" default="0.106871" />
+  <xacro:arg name="thermal_mount_y" default="0.068" />
+  <xacro:arg name="thermal_mount_z" default="0.106136" />
+  <xacro:arg name="thermal_mount_roll" default="0" />
+  <xacro:arg name="thermal_mount_pitch" default="0" />
+  <xacro:arg name="thermal_mount_yaw" default="0" />
   <xacro:property name="simulation_mode" value="$(arg simulation_mode)" />
   <xacro:property name="visualize_sensors" value="$(arg visualize_sensors)" />
@@ -298,8 +307,23 @@
     </collision>
   </link>
+  <!--
+    Mounted beside the RGB-D unit, not in front of it and not on top.
+    On top does not fit: the LiDAR scan plane is at base_link z 0.14712 and the
+    camera body already reaches 0.1197, so a 38 mm board stacked above it tops
+    out at 0.158 and cuts the forward sector of the scan.
+    Beside keeps everything below the scan plane (0.087 - 0.125) and leaves the
+    two optical frames coplanar in x and z, so the baseline is a pure sideways
+    68 mm - the case the thermal-to-RGB calibration is easiest to sanity-check
+    against. The board sits 4 mm clear of the camera housing and 6.5 mm outside
+    the chassis edge, well inside the 0.155 m nav footprint half-width.
+    The three offsets are arguments so the mount can be perturbed by a known
+    amount to test whether a calibration run recovers it.
+  -->
   <joint name="thermal_camera_joint" type="fixed">
     <parent link="base_link" />
     <child link="thermal_camera_link" />
-    <origin xyz="0.158 0 0.112" />
+    <origin
+      xyz="$(arg thermal_mount_x) $(arg thermal_mount_y) $(arg thermal_mount_z)"
+      rpy="$(arg thermal_mount_roll) $(arg thermal_mount_pitch) $(arg thermal_mount_yaw)" />
   </joint>
   <link name="thermal_camera_optical_frame" />

Commit message: feat(calibration): 열화상 외부파라미터를 URDF에 적용
tools/apply_calibration.py 가 캘리브레이션 결과 JSON 을 읽어
config/thermal_extrinsic.yaml 로 쓰고, simulation.launch.py 가 그 파일이
있으면 xacro 인자로 넘깁니다. 보정값은 마운트가 아니라 광학 조인트에
씁니다. 마운트를 옮기면 Fortress 가 렌더하는 카메라도 같이 움직여 보정이
제 꼬리를 물기 때문입니다. 파일을 지우면 도면 기본값으로 돌아갑니다.
열화상 3D 지도가 내부 파라미터를 쓰므로 thermal_camera_info.py 는
simulation.launch.py 가 항상 띄웁니다.

File: src/hazard_guard_simulation/urdf/hazard_guard_m1.urdf.xacro (robot description, xacro)
@@ -23,4 +23,20 @@
   <xacro:arg name="thermal_mount_pitch" default="0" />
   <xacro:arg name="thermal_mount_yaw" default="0" />
+  <!-- Where the thermal optical centre sits inside its own housing. The
+       defaults are the drawing: 9 mm behind the lens face, no rotation beyond
+       the optical convention. Calibration corrects these rather than the mount
+       above, because the mount is the bracket - it carries the visual and the
+       collision, and in Fortress it is also where the sensor renders from,
+       since no <sensor> block carries a <pose>. Moving the bracket to absorb a
+       measured extrinsic would move the rendered camera by the same amount and
+       the correction would chase itself. The optical joint is downstream of
+       the renderer and upstream of TF, which is exactly the seam a calibration
+       belongs in. tools/apply_calibration.py writes these. -->
+  <xacro:arg name="thermal_optical_x" default="0.009" />
+  <xacro:arg name="thermal_optical_y" default="0" />
+  <xacro:arg name="thermal_optical_z" default="0" />
+  <xacro:arg name="thermal_optical_roll" default="-1.57079632679" />
+  <xacro:arg name="thermal_optical_pitch" default="0" />
+  <xacro:arg name="thermal_optical_yaw" default="-1.57079632679" />
   <xacro:property name="simulation_mode" value="$(arg simulation_mode)" />
   <xacro:property name="visualize_sensors" value="$(arg visualize_sensors)" />
@@ -331,5 +347,7 @@
     <parent link="thermal_camera_link" />
     <child link="thermal_camera_optical_frame" />
-    <origin xyz="0.009 0 0" rpy="-1.57079632679 0 -1.57079632679" />
+    <origin
+      xyz="$(arg thermal_optical_x) $(arg thermal_optical_y) $(arg thermal_optical_z)"
+      rpy="$(arg thermal_optical_roll) $(arg thermal_optical_pitch) $(arg thermal_optical_yaw)" />
   </joint>
   <xacro:if value="$(arg include_dispenser)">
